File: NE555_modern/NE555_modern.kicad_sch (KiCad schematic)
At the start: 13 parts, among them SW1 SW_MEC_5G, U1 NE555D

Commit message: 20221221_184000
Parts:
- added J1: Rotrics DexARM, symbol Connector:Conn_01x05_Female
- added J2: Универсальный разъем модуля, symbol Connector:Conn_01x05_Male
Connections:
- net GND: now also J1.5 (Pin_5), J2.5 (Pin_5)
- new net +5V: J1.1 (Pin_1), J2.1 (Pin_1)
- new net Analog: J1.3 (Pin_3), J2.3 (Pin_3)
- new net RX: J1.4 (Pin_4), J2.2 (Pin_2)
- new net TX: J1.2 (Pin_2), J2.4 (Pin_4)
Other:
- note added: "Передача данных"
